Commit message: Add files via upload

File: fanuc/urdf/fanuc.urdf (robot description, URDF)
Before this commit: robot fanuc, 18 links, 17 joints
Links:
- link EE_Base: geometry collision mesh filename=file://$(find fanuc)/urdf/mesh/end_effector.stl scale=0.001 0.001 0.001; visual mesh filename=file://$(find fanuc)/urdf/mesh/end_effector.stl scale=0.001 0.001 0.001
- link Fixed_Base: geometry collision mesh filename=file://$(find fanuc)/urdf/mesh/fixed_base.stl scale=0.001 0.001 0.001; visual mesh filename=file://$(find fanuc)/urdf/mesh/fixed_base.stl scale=0.001 0.001 0.001
- link J1_Upper: geometry collision mesh filename=file://$(find fanuc)/urdf/mesh/upper_link.stl scale=0.001 0.001 0.001; visual mesh filename=file://$(find fanuc)/urdf/mesh/upper_link.stl scale=0.001 0.001 0.001
- link J2_Upper: geometry collision mesh filename=file://$(find fanuc)/urdf/mesh/upper_link.stl scale=0.001 0.001 0.001; visual mesh filename=file://$(find fanuc)/urdf/mesh/upper_link.stl scale=0.001 0.001 0.001
- link J3_Upper: geometry collision mesh filename=file://$(find fanuc)/urdf/mesh/upper_link.stl scale=0.001 0.001 0.001; visual mesh filename=file://$(find fanuc)/urdf/mesh/upper_link.stl scale=0.001 0.001 0.001
