Commit message: Updated urdf file links and robot mesh files

File: fanuc_m430ia/fanuc_m430ia_support/urdf/m430ia.urdf (robot description, URDF)
Before this commit: robot fanuc_m430ia, 9 links, 8 joints
Links:
- added link ee_base; collision mesh filename=package://fanuc_m430ia_support/meshes/gripper/end_effector.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 scale=0.001 0.001 0.001; visual mesh filename=package://fanuc_m430ia_support/meshes/gripper/end_effector.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 scale=0.001 0.001 0.001
- added link left_finger; collision mesh filename=package://fanuc_m430ia_support/meshes/gripper/finger.stl scale=0.001 0.001 0.001; visual mesh filename=package://fanuc_m430ia_support/meshes/gripper/finger.stl scale=0.001 0.001 0.001
- added link right_finger; collision mesh filename=package://fanuc_m430ia_support/meshes/gripper/finger.stl scale=0.001 0.001 0.001; visual mesh filename=package://fanuc_m430ia_support/meshes/gripper/finger.stl scale=0.001 0.001 0.001
- link base_link: geometry collision mesh filename=package://fanuc_m430ia_support/meshes/m430ia/visual/base.stl scale=0.1 0.1 0.1; visual mesh filename=package://fanuc_m430ia_support/meshes/m430ia/visual/base.stl scale=0.1 0.1 0.1
- link link_3: geometry collision mesh filename=package://fanuc_m430ia_support/meshes/m430ia/visual/link_3.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 scale=0.1 0.1 0.1; visual mesh filename=package://fanuc_m430ia_support/meshes/m430ia/visual/link_3.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 scale=0.1 0.1 0.1
Joints:
- added joint ee_base: type fixed, parent flange, child ee_base, origin xyz=0 0 0 rpy=0 0 0
- added joint left_finger: type prismatic, parent ee_base, child left_finger, origin xyz=0 0 0 rpy=0 0 0, axis 0 0 1, limit lower=-0.005 upper=0.02 effort=0 velocity=5
- added joint right_finger: type prismatic, parent ee_base, child right_finger, origin xyz=0 0 0 rpy=0 0 0, axis 0 0 1, limit lower=-0.02 upper=0.005 effort=0 velocity=5
- joint base_link-base: origin xyz=0 0 0.440 rpy=0 0 0 -> xyz=0 0 0.475 rpy=0 0 0
- joint joint_1: origin xyz=0 0 0.440 rpy=0 0 0 -> xyz=0 0 0.475 rpy=0 0 0

File: fanuc_m430ia/fanuc_m430ia_support/urdf/m430ia_macro.xacro (robot description, xacro)
@@ -3,17 +3,17 @@
   <xacro:include filename="$(find fanuc_resources)/urdf/common_materials.xacro"/>
   <xacro:macro name="fanuc_m430ia" params="prefix">
-    <!-- links: main serial chain -->
+    <!-- ~~~~~~~~~~~~~~ LINKS ~~~~~~~~~~~~~~ -->
     <link name="${prefix}base_link">
       <visual>
         <origin xyz="0 0 0" rpy="0 0 0"/>
         <geometry>
-          <mesh filename="package://fanuc_m430ia_support/meshes/m430ia/visual/base_link.stl"/>
-        </geometry>
-        <xacro:material_fanuc_white />
-      </visual>
-      <collision>
-        <origin xyz="0 0 0" rpy="0 0 0"/>
-        <geometry>
-          <mesh filename="package://fanuc_m430ia_support/meshes/m430ia/collision/base_link.stl"/>
+          <mesh filename="package://fanuc_m430ia_support/meshes/m430ia/visual/base.stl" scale="0.1 0.1 0.1"/>
+        </geometry>
+        <xacro:material_fanuc_white />
+      </visual>
+      <collision>
+        <origin xyz="0 0 0" rpy="0 0 0"/>
+        <geometry>
+          <mesh filename="package://fanuc_m430ia_support/meshes/m430ia/collision/base.stl" scale="0.1 0.1 0.1"/>
         </geometry>
       </collision>
@@ -53,12 +53,12 @@
         <origin xyz="0 0 0" rpy="0 0 0"/>
         <geometry>
-          <mesh filename="package://fanuc_m430ia_support/meshes/m430ia/visual/link_3.stl"/>
-        </geometry>
-        <xacro:material_fanuc_white />
-      </visual>
-      <collision>
-        <origin xyz="0 0 0" rpy="0 0 0"/>
-        <geometry>
-          <mesh filename="package://fanuc_m430ia_support/meshes/m430ia/collision/link_3.stl"/>
+          <mesh filename="package://fanuc_m430ia_support/meshes/m430ia/visual/link_3.stl" scale="0.1 0.1 0.1"/>
+        </geometry>
+        <xacro:material_fanuc_white />
+      </visual>
+      <collision>
+        <origin xyz="0 0 0" rpy="0 0 0"/>
+        <geometry>
+          <mesh filename="package://fanuc_m430ia_support/meshes/m430ia/collision/link_3.stl" scale="0.1 0.1 0.1"/>
         </geometry>
       </collision>
@@ -94,65 +94,127 @@
       </collision>
     </link>
-    <!-- joints: main serial chain -->
+    <!-- ~~~~~~~~~~~~~ JOINTS ~~~~~~~~~~~~~~ -->
     <joint name="${prefix}joint_1" type="revolute">
-      <origin xyz="0 0 0.440" rpy="0 0 0"/>
+      <limit lower="-3.1415" upper="3.1415" effort="0" velocity="5.24"/>
+      <origin rpy="0 0 0" xyz="0 0 0.475"/>
       <parent link="${prefix}base_link"/>
       <child link="${prefix}link_1"/>
       <axis xyz="0 0 1"/>
-      <limit lower="-3.1415" upper="3.1415" effort="0" velocity="5.24"/>
     </joint>
     <joint name="${prefix}joint_2" type="revolute">
-      <origin xyz="0 0 0" rpy="0 0 0"/>
+      <limit lower="-2.01" upper="2.01" effort="0" velocity="5.59"/>
+      <origin rpy="0 0 0" xyz="0 0 0"/>
       <parent link="${prefix}link_1"/>
       <child link="${prefix}link_2"/>
       <axis xyz="0 1 0"/>
-      <limit lower="-2.01" upper="2.01" effort="0" velocity="5.59"/>
     </joint>
     <joint name="${prefix}joint_3" type="revolute">
-      <origin xyz="0 -0.095 0.350" rpy="0 0 0"/>
+      <limit lower="-3.34" upper="3.34" effort="0" velocity="5.59"/>
+      <origin rpy="0 0 0" xyz="0 -0.095 0.350"/>
       <parent link="${prefix}link_2"/>
       <child link="${prefix}link_3"/>
       <axis xyz="0 1 0"/>
-      <limit lower="-3.34" upper="3.34" effort="0" velocity="5.59"/>
     </joint>
     <joint name="${prefix}joint_4" type="revolute">
-      <origin xyz="0 0 0.550" rpy="0 0 0"/>
+      <limit lower="-2.62" upper="2.62" effort="0" velocity="6.28"/>
+      <origin rpy="0 0 0" xyz="0 0 0.550"/>
       <parent link="${prefix}link_3"/>
       <child link="${prefix}link_4"/>
       <axis xyz="0 1 0"/>
-      <limit lower="-2.62" upper="2.62" effort="0" velocity="6.28"/>
     </joint>
     <joint name="${prefix}joint_5" type="revolute">
-      <origin xyz="0 0 0.065" rpy="0 0 0"/>
+      <limit lower="-4.71" upper="4.71" effort="0" velocity="20.94"/>
+      <origin rpy="0 0 0" xyz="0 0 0.065"/>
       <parent link="${prefix}link_4"/>
       <child link="${prefix}link_5"/>
       <axis xyz="0 0 1"/>
-      <limit lower="-4.71" upper="4.71" effort="0" velocity="20.94"/>
-    </joint>
-    <!-- ROS-Industrial 'base' frame: base_link to Fanuc World Coordinates transform -->
-    <link name="${prefix}base" />
-    <joint name="${prefix}base_link-base" type="fixed">
-      <origin xyz="0 0 0.440" rpy="0 0 0"/>
-      <parent link="${prefix}base_link"/>
-      <child link="${prefix}base"/>
-    </joint>
-    <!-- ROS-Industrial 'flange' frame: attachment point for EEF models -->
-    <link name="${prefix}flange" />
-    <joint name="${prefix}joint_5-flange" type="fixed">
-      <origin xyz="0 0 0" rpy="0 ${-pi/2.0} 0" />
-      <parent link="${prefix}link_5" />
-      <child link="${prefix}flange" />
-    </joint>
-    <!-- ROS-Industrial 'tool0' frame: all-zeros tool frame -->
-    <link name="${prefix}tool0" />
-    <!-- Note: instead of 'flange', we use 'link_5' as parent of this frame
-               as it already has the correct orientation and location for
-               'tool0'. Using 'flange' here would require additional rotations
-               to undo the rotation introduced by 'joint_5-flange'.
-     -->
-    <joint name="${prefix}link_5-tool0" type="fixed">
-      <origin xyz="0 0 0" rpy="0 0 0" />
-      <parent link="${prefix}link_5" />
-      <child link="${prefix}tool0" />
+    </joint>
+    <!-- ~~~~~~~~~~~~~ CONNECT ~~~~~~~~~~~~~ -->
+    <!-- Base link to work frame -->
+    <link name="base"/>
+    <joint name="base_link-base" type="fixed">
+      <origin rpy="0 0 0" xyz="0 0 0.475"/>
+      <parent link="base_link"/>
+      <child link="base"/>
+    </joint>
+    <!-- Flange attachment point for EEF models -->
+    <link name="flange"/>
+    <joint name="joint_5-flange" type="fixed">
+      <origin rpy="0 -1.5707963267948966 0" xyz="0 0 0"/>
+      <parent link="link_5"/>
+      <child link="flange"/>
+    </joint>
+    <!-- Tool for all-zeros frame -->
+    <link name="tool0"/>
+    <!-- Used instead of flange becuase link is already in correct orientation and location -->
+    <joint name="link_5-tool0" type="fixed">
+      <origin rpy="0 0 0" xyz="0 0 0"/>
+      <parent link="link_5"/>
+      <child link="tool0"/>
+    </joint>
+    <!-- ~~~~~~~~~~~ END EFFECTOR ~~~~~~~~~~ -->
+    <link name="ee_base">
+      <visual>
+        <origin rpy="0 1.5708 0" xyz="0 0 0"/>
+        <geometry>
+          <mesh filename="package://fanuc_m430ia_support/meshes/gripper/end_effector.stl" scale="0.001 0.001 0.001"/>
+        </geometry>
+        <xacro:material_fanuc_white />
+      </visual>
+      <collision>
+        <origin rpy="0 1.5708 0" xyz="0 0 0"/>
+        <geometry>
+          <mesh filename="package://fanuc_m430ia_support/meshes/gripper/end_effector.stl" scale="0.001 0.001 0.001"/>
+        </geometry>
+      </collision>
+    </link>
+    <joint name="ee_base" type="fixed">
+      <origin rpy="0 0 0" xyz="0 0 0"/>
+      <parent link="flange"/>
+      <child link="ee_base"/>
+    </joint>
+    <link name="left_finger">
+      <visual>
+        <origin rpy="-1.5708 0 -1.5708" xyz="0.015 0 0.01"/>
+        <geometry>
+          <mesh filename="package://fanuc_m430ia_support/meshes/gripper/finger.stl" scale="0.001 0.001 0.001"/>
+        </geometry>
+        <xacro:material_fanuc_white />
+      </visual>
+      <collision>
+        <origin rpy="-1.5708 0 -1.5708" xyz="0.015 0 0.01"/>
+        <geometry>
+          <mesh filename="package://fanuc_m430ia_support/meshes/gripper/finger.stl" scale="0.001 0.001 0.001"/>
+        </geometry>
+      </collision>
+    </link>
+    <joint name="left_finger" type="prismatic">
+      <limit lower="-0.005" upper="0.02" effort="0" velocity="5"/>
+      <origin rpy="0 0 0" xyz="0 0 0"/>
+      <parent link="ee_base"/>
+      <child link="left_finger"/>
+      <axis xyz="0 0 1"/>
+    </joint>
+    <link name="right_finger">
+      <visual>
+        <origin rpy="1.5708 0 1.5708" xyz="0.015 0 -0.01"/>
+        <geometry>
+          <mesh filename="package://fanuc_m430ia_support/meshes/gripper/finger.stl" scale="0.001 0.001 0.001"/>
+        </geometry>
+        <xacro:material_fanuc_white />
+      </visual>
+      <collision>
+        <origin rpy="1.5708 0 1.5708" xyz="0.015 0 -0.01"/>
+        <geometry>
+          <mesh filename="package://fanuc_m430ia_support/meshes/gripper/finger.stl" scale="0.001 0.001 0.001"/>
+        </geometry>
+      </collision>
+    </link>
+    <joint name="right_finger" type="prismatic">
+      <limit lower="-0.02" upper="0.005" effort="0" velocity="5"/>
+      <origin rpy="0 0 0" xyz="0 0 0"/>
+      <parent link="ee_base"/>
+      <child link="right_finger"/>
+      <axis xyz="0 0 1"/>
     </joint>
   </xacro:macro>

Commit message: Combined changes

File: fanuc_m430ia/fanuc_m430ia_support/urdf/m430ia.urdf (robot description, URDF)
Before this commit: robot fanuc_m430ia, 12 links, 11 joints
Links:
- added link ee_frame, mass 0.1; collision sphere radius=0.00001; visual sphere radius=0.00001
- link base_link: mass None -> 0.1
- link ee_base: mass None -> 0.1
- link left_finger: mass None -> 0.1
- link link_1: mass None -> 0.1
- link link_2: mass None -> 0.1
- link link_3: mass None -> 0.1
- link link_4: mass None -> 0.1
- link link_5: mass None -> 0.1
- link right_finger: mass None -> 0.1
Joints:
- added joint ee_frame: type fixed, parent ee_base, child ee_frame, origin xyz=0 0 0.055 rpy=0 0 0
- added joint world_fixture: type fixed, parent world, child base_link
- joint base_link-base: origin xyz=0 0 0.475 rpy=0 0 0 -> xyz=0 0 0.440 rpy=0 0 0
- joint joint_1: limit lower=-3.1415 upper=3.1415 effort=0 velocity=5.24 -> lower=-3.1415 upper=3.1415 effort=30 velocity=5.24; origin xyz=0 0 0.475 rpy=0 0 0 -> xyz=0 0 0.440 rpy=0 0 0
- joint joint_2: limit lower=-2.01 upper=2.01 effort=0 velocity=5.59 -> lower=-2.01 upper=2.01 effort=30 velocity=5.59
- joint joint_3: limit lower=-3.34 upper=3.34 effort=0 velocity=5.59 -> lower=-3.34 upper=3.34 effort=30 velocity=5.59
- joint joint_4: limit lower=-2.62 upper=2.62 effort=0 velocity=6.28 -> lower=-2.62 upper=2.62 effort=30 velocity=6.28
- joint joint_5: limit lower=-4.71 upper=4.71 effort=0 velocity=20.94 -> lower=-4.71 upper=4.71 effort=30 velocity=20.94
- joint joint_5-flange: origin xyz=0 0 0 rpy=0 -1.5707963267948966 0 -> xyz=0 0 0 rpy=0 0 0
- joint left_finger: axis 0 0 1 -> 1 0 0
- joint link_5-tool0: origin xyz=0 0 0 rpy=0 0 0 -> xyz=0 0 0 rpy=0 1.5708 0
- joint right_finger: axis 0 0 1 -> 1 0 0; mimic (none) -> joint=left_finger multiplier=-1 offset=0

Commit message: Updated to use both fingers

File: fanuc_m430ia/fanuc_m430ia_support/urdf/m430ia.urdf (robot description, URDF)
Before this commit: robot fanuc_m430ia, 14 links, 13 joints
Links:
- removed link base
- link ee_frame: mass 0.1 -> 0.01
- link left_finger: mass 0.1 -> 0.01
- link right_finger: mass 0.1 -> 0.01
Joints:
- removed joint base_link-base
- removed joint left_finger
- removed joint right_finger
- added joint left_finger_joint: type prismatic, parent ee_base, child left_finger, origin xyz=0 0 0 rpy=0 0 0, axis 1 0 0, limit lower=-0.005 upper=0.02 effort=10 velocity=5
- added joint right_finger_joint: type prismatic, parent ee_base, child right_finger, origin xyz=0 0 0 rpy=0 0 0, axis 1 0 0, limit lower=-0.02 upper=0.005 effort=10 velocity=5
